File: hardware/MP3 Shield.sch (EAGLE design)
At the start: 52 parts, among them Q1 12.288MHz, U1 3.3V, U2 ARDUINO_SHIELD, U3 VS1053, U4 1.8V, U6 USD-SOCKET, U7 74HC4050 LVL CONVERTER

Commit message: More WIP.
Parts:
- removed SJ1: NC, SparkFun:SOLDERJUMPERTRACE
- removed U$7: LOGO-SFENEW, SparkFun:LOGO-SFENEW
- removed U5: (no value), SparkFun:AUDIO-JACKSMD2
- added C17, C18: 10uF, SparkFun-Capacitors:10UF-16V-10%(TANT)
- added C19, C20: 3.3nF, SparkFun-Capacitors:3.3NF-100V-10%(0603)
- added J1: ISP/SPI, SparkFun:AVR_SPI_PRG_6PTH
- added LOGO1: OSHW-LOGOS, SparkFun-Aesthetics:OSHW-LOGOS
- added LOGO2: SFE_LOGO_NAME_FLAME.1_INCH, SparkFun-Aesthetics:SFE_LOGO_NAME_FLAME.1_INCH
- added R15, R16: 10K, SparkFun-Resistors:10KOHM1/10W1%(0603)0603
- added R21, R22: 470, SparkFun-Resistors:470OHM1/10W1%(0603)
- added R23: 1K, SparkFun-Resistors:1KOHM1/10W1%(0603)
- added SJ3, SJ4: NC, SparkFun:SOLDERJUMPERTRACE
- added SJ7, SJ8, SJ9: JUMPER-PAD-3-2OF3_NC_BY_TRACE, SparkFun-Passives:JUMPER-PAD-3-2OF3_NC_BY_TRACE
- C1, C6: device SparkFun:CAP_POL1206 -> SparkFun-Capacitors:10UF-16V-10%(TANT)
- C10, C11: device SparkFun:CAP0402-CAP -> SparkFun-Capacitors:10NF/10000PF-50V-10%(0603)
- C12: device SparkFun:CAP0402-CAP -> SparkFun-Capacitors:47NF(0.047UF/47000PF)-25V-5%(0603)SMD
- C13, C14, C15, C16, C2, C5, C7: device SparkFun:CAP0402-CAP -> SparkFun-Capacitors:0.1UF-25V(+80/-20%)(0603)
- C3, C8: device SparkFun:CAP0402-CAP -> SparkFun-Capacitors:22PF-50V-5%(0603)
- C4: device SparkFun:CAP0402-CAP -> SparkFun-Capacitors:470PF-50V-5%(0603)SMD
- C9: device SparkFun:CAP0402-CAP -> SparkFun-Capacitors:1.0UF-16V-10%(0603)
- JP1: value Line Output -> (none); device SparkFun:M03PTH -> SparkFun-Connectors:AUDIO-JACKSMD2
- JP3: value External Speaker -> Optional
- LED1: device SparkFun:LED0603 -> SparkFun-LED:LED-RED0603
- R1: device SparkFun:RESISTOR0402-RES -> SparkFun-Resistors:1M-1%
- R10, R11, R12, R2, R3, R4, R5: device SparkFun:RESISTOR0402-RES -> SparkFun-Resistors:100KOHM1/10W1%(0603)
- R13, R14: device SparkFun:RESISTOR0402-RES -> SparkFun-Resistors:1KOHM1/10W1%(0603)
- R6, R7: device SparkFun:RESISTOR0402-RES -> SparkFun-Resistors:20OHM1/10W1%(0603)SMD
- R8: device SparkFun:RESISTOR0402-RES -> SparkFun-Resistors:330OHM1/10W1%(0603)
- R9: device SparkFun:RESISTOR0402-RES -> SparkFun-Resistors:10OHM1/10W5%0603SMD
- S2: device SparkFun:SWITCH-MOMENTARY-2SMD -> SparkFun-Electromechanical:SWITCH-MOMENTARY-2SMD
- U1: device SparkFun:V_REG_LDOSMD -> SparkFun-PowerIC:V_REG_MIC52053.3V
- U2: value ARDUINO_SHIELD -> ARDUINO_R3_SHIELD; device SparkFun:ARDUINO_SHIELDLABEL -> SparkFun-Boards:ARDUINO_R3_SHIELD
- U3: device SparkFun:VS1033 -> SparkFun-DigitalIC:VS1033/1053SMD
- U4: device SparkFun:V_REG_LDOSMD2 -> SparkFun-PowerIC:V_REG_SP62141.8V
- U7: device SparkFun:HEX_CONVERTER -> SparkFun-DigitalIC:HEX_CONVERTER
Connections:
- net N$1 renamed RCAP
- net N$73 renamed GPIO4
- new net /MUTE: R23.1
- new net 5V-MUTE: SJ4.2, U2.*D5
- new net N$14: R23.2, SJ4.1
- new net N$17: C18.+, C20.1, R22.1
- new net N$19: C17.+, C19.1, R21.1
- new net SPKR-L: C17.-, R15.1
- new net SPKR-R: C18.-, R16.1
- net 3.3V: no longer R5.1
- net 5V-GPIO1: now also SJ3.2; no longer SJ1.2
- net 5V-MOSI: now also J1.4
- net 5V-SCK: now also J1.3
- net GBUF: no longer JP3.1, U5.SLEEVE
- net GND: now also C19.2, C20.2, J1.6, R15.2, R16.2, R5.1, SJ9.1
- net LEFT: now also R21.2; no longer JP3.3, U5.LEFT
- net MISO: now also J1.1
- net N$4: now also SJ3.1; no longer SJ1.1
- net RIGHT: now also R22.2; no longer JP3.2, U5.RIGHT
- net VCC: now also J1.2
Other:
- note added: "150mA"
- note added: "Added MUTE"
- note added: "Added OSHW mark"
- note added: "Added solder jumper to select between GBUF and GND"
- note added: "Added transient free line-out connection"
- note added: "Arduino"
- note added: "Changed all 0402 footprints to 0603 for easier optical inspection"
- note added: "Connect GBUF if attaching amplifier"
- note added: "Connect GND if attaching external speakers (default)"
- note added: "Line Out to Speakers or Amplifier"
- note added: "Moved to tighter SOIC FP on HEX inverter"
- note added: "New on v1.4:"
- note added: "Populate with 2x3 female connector to be compatible with Leonardo/Mega"
- note added: "RST now pulled low by default"
- note added: "Solder Jumper 3:"
- note added: "Touched up 3.5mm jack footprint"
- note added: "Update to Arduino R3 shield type"
- note added: "Updated version code"
- note added: "v1.5"
- note removed: "Arduino Shield Footprint"
- note removed: "Outputs"
- note removed: "V1.5"
- moved on the sheet: C1, C10, C11, C12, C13, C14, C15, C16, C2, C3, C4, C5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

Commit message: Yet more WIP
Parts:
- removed R23: 1K, SparkFun-Resistors:1KOHM1/10W1%(0603)
- removed SJ8, SJ9: JUMPER-PAD-3-2OF3_NC_BY_TRACE, SparkFun-Passives:JUMPER-PAD-3-2OF3_NC_BY_TRACE
- added SJ1: NC, SparkFun:SOLDERJUMPERTRACE
- SJ3: value NC -> AC Coupling Gnd; device SparkFun:SOLDERJUMPERTRACE -> SparkFun-Passives:JUMPER-PAD-3-2OF3_NC_BY_TRACE
- SJ4: value NC -> AC Coupling R; device SparkFun:SOLDERJUMPERTRACE -> SparkFun-Passives:JUMPER-PAD-3-2OF3_NC_BY_TRACE
- SJ5: value JUMPER-PAD-3-2OF3_NC_BY_TRACE -> AC Coupling L
- renumbered SJ7 to SJ5
Connections:
- removed net /MUTE: R23.1
- removed net 5V-MUTE: SJ4.2, U2.*D5
- new net N$12: JP1.SLEEVE, JP3.1, SJ3.2
- new net N$13: JP1.RIGHT, JP3.2, SJ4.2
- net 5V-GPIO1: now also SJ1.2; no longer SJ3.2
- net GBUF: now also SJ3.3
- net GND: now also SJ3.1; no longer SJ9.1
- net LEFT: now also SJ5.3
- net N$14: now also JP1.LEFT, JP3.3, SJ5.2; no longer R23.2, SJ4.1
- net N$4: now also SJ1.1; no longer SJ3.1
- net RIGHT: now also SJ4.3
- net SPKR-L: now also SJ5.1
- net SPKR-R: now also SJ4.1
Other:
- note added: "Leave at default connection for DC-coupled output to headphones or passive speakers. Cut default and add solder blob to bottom pads for AC-coupled line output."
- note added: "Solder Jumpers 3, 4, 5:"
- note removed: "Connect GBUF if attaching amplifier"
- note removed: "Connect GND if attaching external speakers (default)"
- note removed: "Solder Jumper 3:"
- moved on the sheet: JP1, JP3

Commit message: V1.5 ready for protos.
Board routed and ready for protos.
Parts:
- removed C19, C20: 3.3nF, SparkFun-Capacitors:3.3NF-100V-10%(0603)
- SJ3, SJ4, SJ5: device SparkFun-Passives:JUMPER-PAD-3-2OF3_NC_BY_TRACE -> SparkFun-Passives:JUMPER-PAD-3-2OF3_NC_BY_PASTE
Connections:
- net GND: no longer C19.2, C20.2
- net N$17: no longer C20.1
- net N$19: no longer C19.1
Changed lines of the file:
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@@
 <part name="C17" library="SparkFun-Capacitors" deviceset="10UF-16V-10%(TANT)" device="" value="10uF"/>
 <part name="C18" library="SparkFun-Capacitors" deviceset="10UF-16V-10%(TANT)" device="" value="10uF"/>
-<part name="C19" library="SparkFun-Capacitors" deviceset="3.3NF-100V-10%(0603)" device="" value="3.3nF"/>
-<part name="C20" library="SparkFun-Capacitors" deviceset="3.3NF-100V-10%(0603)" device="" value="3.3nF"/>
-<part name="GND30" library="SparkFun" deviceset="GND" device=""/>
 <part name="GND31" library="SparkFun" deviceset="GND" device=""/>
 <part name="GND32" library="SparkFun" deviceset="GND" device=""/>
 <part name="GND37" library="SparkFun" deviceset="GND" device=""/>
 <part name="GND38" library="SparkFun" deviceset="GND" device=""/>
-<part name="GND39" library="SparkFun" deviceset="GND" device=""/>
 <part name="GND33" library="SparkFun" deviceset="GND" device=""/>
 <part name="FRAME1" library="SparkFun-Aesthetics" deviceset="FRAME-LEDGER" device=""/>
@@
 <part name="P+9" library="SparkFun" deviceset="VCC" device=""/>
 <part name="U$1" library="SparkFun-Aesthetics" deviceset="REVISION" device=""/>
-<part name="SJ5" library="SparkFun-Passives" deviceset="JUMPER-PAD-3-2OF3_NC_BY_TRACE" device="" value="AC Coupling L"/>
-<part name="SJ4" library="SparkFun-Passives" deviceset="JUMPER-PAD-3-2OF3_NC_BY_TRACE" device="" value="AC Coupling R"/>
-<part name="SJ3" library="SparkFun-Passives" deviceset="JUMPER-PAD-3-2OF3_NC_BY_TRACE" device="" value="AC Coupling Gnd"/>
+<part name="SJ5" library="SparkFun-Passives" deviceset="JUMPER-PAD-3-2OF3_NC_BY_PASTE" device="" value="AC Coupling L"/>
+<part name="SJ4" library="SparkFun-Passives" deviceset="JUMPER-PAD-3-2OF3_NC_BY_PASTE" device="" value="AC Coupling R"/>
+<part name="SJ3" library="SparkFun-Passives" deviceset="JUMPER-PAD-3-2OF3_NC_BY_PASTE" device="" value="AC Coupling Gnd"/>
 <part name="GND29" library="SparkFun" deviceset="GND" device=""/>
 </parts>
@@
 <instance part="C17" gate="G$1" x="294.64" y="162.56" rot="MR270"/>
 <instance part="C18" gate="G$1" x="294.64" y="129.54" rot="MR270"/>
-<instance part="C19" gate="G$1" x="284.48" y="154.94"/>
-<instance part="C20" gate="G$1" x="284.48" y="121.92"/>
-<instance part="GND30" gate="1" x="284.48" y="147.32"/>
 <instance part="GND31" gate="1" x="304.8" y="144.78"/>
 <instance part="GND32" gate="1" x="304.8" y="111.76"/>
 <instance part="GND37" gate="1" x="269.24" y="60.96" rot="MR0"/>
 <instance part="GND38" gate="1" x="269.24" y="134.62" rot="MR0"/>
-<instance part="GND39" gate="1" x="284.48" y="114.3"/>
 <instance part="GND33" gate="1" x="195.58" y="114.3"/>
 <instance part="FRAME1" gate="G$1" x="0" y="0"/>
@@
 </segment>
 <segment>
-<pinref part="C20" gate="G$1" pin="2"/>
-<pinref part="GND39" gate="1" pin="GND"/>
-<wire x1="284.48" y1="116.84" x2="284.48" y2="119.38" width="0.1524" layer="91"/>
-</segment>
-<segment>
 <pinref part="R15" gate="G$1" pin="2"/>
 <pinref part="GND31" gate="1" pin="GND"/>
 <wire x1="304.8" y1="147.32" x2="304.8" y2="149.86" width="0.1524" layer="91"/>
-</segment>
-<segment>
-<pinref part="C19" gate="G$1" pin="2"/>
-<pinref part="GND30" gate="1" pin="GND"/>
-<wire x1="284.48" y1="149.86" x2="284.48" y2="152.4" width="0.1524" layer="91"/>
 </segment>
 <segment>
@@
 <segment>
 <pinref part="C18" gate="G$1" pin="+"/>
-<pinref part="C20" gate="G$1" pin="1"/>
-<wire x1="292.1" y1="129.54" x2="284.48" y2="129.54" width="0.1524" layer="91"/>
-<wire x1="284.48" y1="129.54" x2="284.48" y2="127" width="0.1524" layer="91"/>
-<wire x1="284.48" y1="129.54" x2="281.94" y2="129.54" width="0.1524" layer="91"/>
-<junction x="284.48" y="129.54"/>
+<wire x1="292.1" y1="129.54" x2="281.94" y2="129.54" width="0.1524" layer="91"/>
 <pinref part="R22" gate="G$1" pin="1"/>
 </segment>
@@
 <pinref part="R21" gate="G$1" pin="1"/>
 <pinref part="C17" gate="G$1" pin="+"/>
-<wire x1="281.94" y1="162.56" x2="284.48" y2="162.56" width="0.1524" layer="91"/>
-<pinref part="C19" gate="G$1" pin="1"/>
-<wire x1="284.48" y1="162.56" x2="292.1" y2="162.56" width="0.1524" layer="91"/>
-<wire x1="284.48" y1="160.02" x2="284.48" y2="162.56" width="0.1524" layer="91"/>
-<junction x="284.48" y="162.56"/>
-</segment>
-</net>
+<wire x1="281.94" y1="162.56" x2="292.1" y2="162.56" width="0.1524" layer="91"/>
+</segment>
+</net>

Commit message: Ready to review for reds
Reorganized the solder jumpers for output coupling selection.
Parts:
- SJ3: value AC Coupling Gnd -> AC Coupling L
- SJ5: value AC Coupling L -> AC Coupling Gnd
Connections:
- net GBUF: now also SJ5.3; no longer SJ3.3
- net GND: now also SJ5.1; no longer SJ3.1
- net LEFT: now also SJ3.3; no longer SJ5.3
- net N$12: now also SJ5.2; no longer SJ3.2
- net N$14: now also SJ3.2; no longer SJ5.2
- net SPKR-L: now also SJ3.1; no longer SJ5.1
Other:
- moved on the sheet: SJ3, SJ5
Changed lines of the file:
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@@
 <part name="P+9" library="SparkFun" deviceset="VCC" device=""/>
 <part name="U$1" library="SparkFun-Aesthetics" deviceset="REVISION" device=""/>
-<part name="SJ5" library="SparkFun-Passives" deviceset="JUMPER-PAD-3-2OF3_NC_BY_PASTE" device="" value="AC Coupling L"/>
+<part name="SJ3" library="SparkFun-Passives" deviceset="JUMPER-PAD-3-2OF3_NC_BY_PASTE" device="" value="AC Coupling L"/>
 <part name="SJ4" library="SparkFun-Passives" deviceset="JUMPER-PAD-3-2OF3_NC_BY_PASTE" device="" value="AC Coupling R"/>
-<part name="SJ3" library="SparkFun-Passives" deviceset="JUMPER-PAD-3-2OF3_NC_BY_PASTE" device="" value="AC Coupling Gnd"/>
+<part name="SJ5" library="SparkFun-Passives" deviceset="JUMPER-PAD-3-2OF3_NC_BY_PASTE" device="" value="AC Coupling Gnd"/>
 <part name="GND29" library="SparkFun" deviceset="GND" device=""/>
 </parts>
@@
 <instance part="P+9" gate="1" x="60.96" y="109.22"/>
 <instance part="U$1" gate="G$1" x="331.47" y="6.858"/>
-<instance part="SJ5" gate="G$1" x="355.6" y="152.4" rot="R180"/>
+<instance part="SJ3" gate="G$1" x="355.6" y="152.4" rot="R180"/>
 <instance part="SJ4" gate="G$1" x="355.6" y="121.92" rot="R180"/>
-<instance part="SJ3" gate="G$1" x="355.6" y="91.44" rot="R180"/>
+<instance part="SJ5" gate="G$1" x="355.6" y="91.44" rot="R180"/>
 <instance part="GND29" gate="1" x="355.6" y="81.28"/>
 </instances>
@@
 <segment>
 <pinref part="GND29" gate="1" pin="GND"/>
-<pinref part="SJ3" gate="G$1" pin="1"/>
+<pinref part="SJ5" gate="G$1" pin="1"/>
 <wire x1="355.6" y1="83.82" x2="355.6" y2="86.36" width="0.1524" layer="91"/>
 </segment>
@@
 <segment>
 <label x="347.98" y="162.56" size="1.27" layer="95" rot="R180" xref="yes"/>
-<pinref part="SJ5" gate="G$1" pin="3"/>
+<pinref part="SJ3" gate="G$1" pin="3"/>
 <wire x1="355.6" y1="157.48" x2="355.6" y2="162.56" width="0.1524" layer="91"/>
 <wire x1="355.6" y1="162.56" x2="347.98" y2="162.56" width="0.1524" layer="91"/>
@@
 <label x="350.52" y="99.06" size="1.27" layer="95" rot="R180" xref="yes"/>
 <wire x1="350.52" y1="99.06" x2="355.6" y2="99.06" width="0.1524" layer="91"/>
-<pinref part="SJ3" gate="G$1" pin="3"/>
+<pinref part="SJ5" gate="G$1" pin="3"/>
 <wire x1="355.6" y1="99.06" x2="355.6" y2="96.52" width="0.1524" layer="91"/>
 </segment>
@@
 <segment>
 <label x="347.98" y="144.78" size="1.27" layer="95" rot="R180" xref="yes"/>
-<pinref part="SJ5" gate="G$1" pin="1"/>
+<pinref part="SJ3" gate="G$1" pin="1"/>
 <wire x1="355.6" y1="147.32" x2="355.6" y2="144.78" width="0.1524" layer="91"/>
 <wire x1="355.6" y1="144.78" x2="347.98" y2="144.78" width="0.1524" layer="91"/>
@@
 <net name="N$12" class="0">
 <segment>
-<pinref part="SJ3" gate="G$1" pin="2"/>
+<pinref part="SJ5" gate="G$1" pin="2"/>
 <wire x1="360.68" y1="91.44" x2="373.38" y2="91.44" width="0.1524" layer="91"/>
 <wire x1="373.38" y1="91.44" x2="373.38" y2="152.4" width="0.1524" layer="91"/>
@@
 <net name="N$14" class="0">
 <segment>
-<pinref part="SJ5" gate="G$1" pin="2"/>
+<pinref part="SJ3" gate="G$1" pin="2"/>
 <wire x1="360.68" y1="152.4" x2="368.3" y2="152.4" width="0.1524" layer="91"/>
 <wire x1="368.3" y1="152.4" x2="368.3" y2="157.48" width="0.1524" layer="91"/>
