File: hardware/SparkFunMP3Shield.sch (EAGLE design)
At the start: 62 parts, among them J1 ISP/SPI, Q1 12.288MHz, U1 3.3V, U2 ARDUINO_R3_SHIELD, U3 VS1053, U4 1.8V, U6 USD-SOCKET, U7 74HC4050 LVL CONVERTER

Commit message: Use traces to close jumpers
Parts:
- SJ3, SJ4, SJ5: device SparkFun-Passives:JUMPER-PAD-3-2OF3_NC_BY_PASTE -> SparkFun-Jumpers:JUMPER-SMT_3_1-NC_TRACE_SILK
